File: hw/54PinTo60RibbonAdapterBoard/54PinTo60RibbonAdapterBoard.kicad_sch (KiCad schematic)
At the start: 3 parts, among them J1 Conn_02x27_Odd_Even, J2 Conn_01x60_Pin, J99 Conn_01x54_MountingPin

Commit message: Updated FPC connector on 54 Pin Adapter Board
Parts:
- J1: now left out of the parts list
- J2: footprint Connector_FFC-FPC:Amphenol_F32R-1A7x1-11060_1x60-1MP_P0.5mm_Horizontal -> gg_lcd:1x54 To 1x60 FPC Connector 0.5mm; now left out of the parts list
Changed lines of the file:
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@@
 		(unit 1)
 		(exclude_from_sim no)
-		(in_bom yes)
+		(in_bom no)
 		(on_board yes)
 		(dnp no)
@@
 			)
 		)
-		(property "Footprint" "Connector_FFC-FPC:Amphenol_F32R-1A7x1-11060_1x60-1MP_P0.5mm_Horizontal"
+		(property "Footprint" "gg_lcd:1x54 To 1x60 FPC Connector 0.5mm"
 			(at 143.51 69.85 0)
 			(effects
@@
 		(unit 1)
 		(exclude_from_sim no)
-		(in_bom yes)
+		(in_bom no)
 		(on_board yes)
 		(dnp no)
